File: rev b/tiny-osean.kicad_pcb (KiCad board)
At the start: 2 copper layers, 65.2 x 65.2 mm, 22 parts, among them J1 VCC, J2 UPDI, J3 GND, SW1 SW_Push, U1 ATtiny816-M

Commit message: started rev b
Parts:
- added D1: Green, Capacitor_SMD:C_0805_2012Metric_Pad1.18x1.45mm_HandSolder, F.Cu at (202.0, 88.0)
- added D2: Green, Capacitor_SMD:C_0805_2012Metric_Pad1.18x1.45mm_HandSolder, F.Cu at (202.0, 85.0)
- added D3: Red, Capacitor_SMD:C_0805_2012Metric_Pad1.18x1.45mm_HandSolder, F.Cu at (206.8, 88.0)
- added D4: Red, Capacitor_SMD:C_0805_2012Metric_Pad1.18x1.45mm_HandSolder, F.Cu at (206.8, 85.0)
- added D5: Blue, Capacitor_SMD:C_0805_2012Metric_Pad1.18x1.45mm_HandSolder, F.Cu at (211.6, 85.0)
- added D6: Blue, Capacitor_SMD:C_0805_2012Metric_Pad1.18x1.45mm_HandSolder, F.Cu at (202.0, 91.0)
- added R10: 10, Resistor_SMD:R_0402_1005Metric, F.Cu at (212.7, 93.5)
- added R11: 10, Resistor_SMD:R_0402_1005Metric, F.Cu at (204.0, 93.5)
- added R12: 10, Resistor_SMD:R_0402_1005Metric, F.Cu at (211.7, 89.5)
- added R13: 10, Resistor_SMD:R_0402_1005Metric, F.Cu at (210.7, 87.5)
- added R14: 10, Resistor_SMD:R_0402_1005Metric, F.Cu at (212.7, 95.5)
- added R15: 10, Resistor_SMD:R_0402_1005Metric, F.Cu at (206.9, 94.5)
- added R16: 10, Resistor_SMD:R_0402_1005Metric, F.Cu at (214.6, 89.5)
- added R17: 10, Resistor_SMD:R_0402_1005Metric, F.Cu at (201.1, 93.5)
- added R18: 10, Resistor_SMD:R_0402_1005Metric, F.Cu at (216.5, 86.5)
- added R19: 10, Resistor_SMD:R_0402_1005Metric, F.Cu at (217.5, 88.5)
- added R2: 10, Resistor_SMD:R_0402_1005Metric, F.Cu at (209.8, 94.5)
- added R20: 10, Resistor_SMD:R_0402_1005Metric, F.Cu at (219.4, 86.5)
- added R21: 10, Resistor_SMD:R_0402_1005Metric, F.Cu at (212.7, 91.5)
- added R22: 10, Resistor_SMD:R_0402_1005Metric, F.Cu at (215.6, 91.5)
- added R23: 10, Resistor_SMD:R_0402_1005Metric, F.Cu at (215.5, 84.5)
- added R24: 10, Resistor_SMD:R_0402_1005Metric, F.Cu at (218.4, 84.5)
- added R25: 10, Resistor_SMD:R_0402_1005Metric, F.Cu at (205.9, 90.5)
- added R3: 10, Resistor_SMD:R_0402_1005Metric, F.Cu at (213.6, 87.5)
- added R4: 10, Resistor_SMD:R_0402_1005Metric, F.Cu at (208.8, 90.5)
- added R5: 10, Resistor_SMD:R_0402_1005Metric, F.Cu at (209.8, 92.5)
- added R6: 10, Resistor_SMD:R_0402_1005Metric, F.Cu at (206.9, 92.5)
- U1: value ATtiny816-M -> ATtiny1616-M
Connections:
- R7 pad 1: Net-(R6-Pad2) -> Net-(R7-Pad1)
- R9 pad 2: Net-(JP2-Pad2) -> PB0
- U1 pad 15: unconnected-(U1-Pad15) -> PC0
- U1 pad 16: unconnected-(U1-Pad16) -> PC1
- U1 pad 5: unconnected-(U1-Pad5) -> PA4
- U1 pad 6: unconnected-(U1-Pad6) -> PA5
Routing:
- net PB0: track 3.36 -> 12.4 mm
- net Net-(JP2-Pad2): track 9.02 -> 0.00 mm
- net Net-(R7-Pad1): track 0.00 -> 1.55 mm
- net Net-(R6-Pad2): track 1.55 -> 0.00 mm

Commit message: finished rev b in one night cause discounts dont last forever
Parts:
- removed the D1 at (155.0, 89.1)
- removed the D2 at (139.0, 106.1)
- removed JP1, JP2: SolderJumper_2_Open, Jumper:SolderJumper-2_P1.3mm_Open_TrianglePad1.0x1.5mm
- removed the R2 at (157.2, 84.6)
- removed the R3 at (158.1, 85.5)
- removed the R4 at (158.9, 86.3)
- removed the R5 at (159.7, 87.2)
- removed the R6 at (134.1, 106.3)
- moved R2 79.3 mm to (135.0, 120.7), turned to -135 degrees
- moved R20 77.5 mm to (145.8, 110.8), turned to 45 degrees
- moved R13 77.3 mm to (134.2, 98.8), turned to 45 degrees
- moved R12 77.3 mm to (135.1, 99.6), turned to -135 degrees
- moved R10 76.4 mm to (136.7, 101.2), turned to -135 degrees
- moved R18 75.7 mm to (144.2, 109.2), turned to 45 degrees
- moved R19 75.6 mm to (145.0, 110.0), turned to -135 degrees
- moved D5 73.0 mm to (141.9, 106.5), turned to 45 degrees
- moved D3 69.2 mm to (139.6, 104.2), turned to 135 degrees
- moved R21 69.1 mm to (146.6, 111.7), turned to -135 degrees
- moved R11 68.4 mm to (135.9, 100.4), turned to 45 degrees
- moved D1 66.4 mm to (138.1, 106.0), turned to 135 degrees
- moved R16 64.8 mm to (150.0, 85.1), turned to 45 degrees
- moved R14 61.6 mm to (151.7, 86.9), turned to 45 degrees
- moved R24 58.8 mm to (160.7, 95.4), turned to 45 degrees
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Routing:
- net VCC: track 103.4 -> 7.58 mm, vias 14 -> 0
- net PA5: track 0.00 -> 52.4 mm
- net PB1: track 5.29 -> 57.4 mm, vias 0 -> 2
- net PC1: track 0.00 -> 44.1 mm, vias 0 -> 2
- net Net-(JP1-Pad2): track 41.0 -> 0.00 mm
- net GND: track 4.53 -> 45.3 mm, vias 1 -> 14
- net PA4: track 0.00 -> 30.4 mm, vias 0 -> 2
- net PC0: track 0.00 -> 27.3 mm
- net Net-(D3-Pad1): track 0.00 -> 11.7 mm
- net Net-(D1-Pad1): track 5.32 -> 15.0 mm
- net PB0: track 12.4 -> 3.50 mm
- net Net-(D4-Pad1): track 0.00 -> 7.62 mm
- net Net-(D6-Pad1): track 0.00 -> 4.07 mm
- net Net-(D5-Pad1): track 0.00 -> 3.65 mm
- net Net-(D2-Pad1): track 5.93 -> 4.56 mm
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- added copper zone on B.Cu, net GND
- added copper zone on F.Cu, net VCC
- removed copper zone on F.Cu, net GND
- removed copper zone on B.Cu, net VCC
Other:
- board text added: "REV B"
- board text removed: "REV A"
